File: Hardware/MiniArmController.kicad_sch (KiCad schematic)
At the start: 7 parts, among them U1 Teensy4.1_DEV-16771

Commit message: Superseded board changes
Parts:
- added C1: 0.1uF, Capacitor_SMD:C_0603_1608Metric_Pad1.08x0.95mm_HandSolder, symbol Device:C
- added C2: 10uF, Capacitor_SMD:C_1206_3216Metric_Pad1.33x1.80mm_HandSolder, symbol Device:C
- added C3: 10uF, Capacitor_SMD:C_0603_1608Metric_Pad1.08x0.95mm_HandSolder, symbol Device:C
- added Conn3: AndersonPP, MRDT_Connectors:Square_Anderson_2_H_Side_By_Side_PV, symbol MRDT_Connectors:AndersonPP
- added J1: RJ45_LED_Shielded, MRDT_Connectors:RJ45_Teensy, symbol Connector:RJ45_LED_Shielded
- added U6: OKI, MRDT_Devices:OKI_Horizontal, symbol MRDT_Devices:OKI
- Conn1, Conn2: footprint (none) -> MRDT_Connectors:MOLEX_SL_03_Vertical
- U1: footprint MODULE_DEV-16771 -> MRDT_Shields:Teensy_4_1
- U4, U5: footprint (none) -> MiniArmController:DIP-16_W12.7mm
Connections:
- net +3V3: now also U4.1 (VIO), U5.1 (VIO); no longer U4.8 (VIO), U5.8 (VIO)
- net +7.5V: now also U4.16 (VIN), U5.16 (VIN); no longer U4.9 (VIN), U5.9 (VIN)
- net GND: now also U4.15 (GND), U4.9 (GND), U5.15 (GND), U5.9 (GND), C1.1, C2.2, C3.2, Conn3.1 (GND), J1.8, J1.9, J1.SH, U6.2 (GND); no longer U4.10 (GND), U4.16 (GND), U5.10 (GND), U5.16 (GND)
- net UH1: now also U5.3 (UH); no longer U5.6 (UH)
- net UH2: now also U4.3 (UH); no longer U4.6 (UH)
- net UL1: now also U5.2 (UL); no longer U5.7 (UL)
- net UL2: now also U4.2 (UL); no longer U4.7 (UL)
- net VH1: now also U5.5 (VH); no longer U5.4 (VH)
- net VH2: now also U4.5 (VH); no longer U4.4 (VH)
- net VL1: now also U5.4 (VL); no longer U5.5 (VL)
- net VL2: now also U4.4 (VL); no longer U4.5 (VL)
- net WH1: now also U5.7 (WH); no longer U5.2 (WH)
- net WH2: now also U4.7 (WH); no longer U4.2 (WH)
- net WL1: now also U5.6 (WL); no longer U5.3 (WL)
- net WL2: now also U4.6 (WL); no longer U4.3 (WL)
- net at Conn2.1: now also U4.14 (U); no longer U4.11 (U)
- net at Conn2.2: now also U4.13 (V); no longer U4.12 (V)
- net at Conn2.3: now also U4.12 (W); no longer U4.13 (W)
- net +5V: now reaches U1.5V
- net +5V: now also C3.1, U6.3 (Vo)
- net at U1.LED: now also J1.10
- net R+: now reaches U1.R+
- net R+: now also J1.4
- net R-: now reaches U1.R-
- net R-: now also J1.6
- net T+: now reaches U1.T+
- net T+: now also J1.1
- net T-: now reaches U1.T-
- net T-: now also J1.3
- net at Conn1.1: now also U5.14 (U); no longer U5.11 (U)
- net at Conn1.2: now also U5.13 (V); no longer U5.12 (V)
- net at Conn1.3: now also U5.12 (W); no longer U5.13 (W)
- new net: C1.2, J1.2, J1.5
- new net PV: C2.1, Conn3.4 (PV+), U6.1 (Vi)
- no-connect marks 10 -> 13
Other:
- note added: "Encoders"
- note added: "Motor Controllers"
- note added: "Power"
- note added: "Teensy"
- moved on the sheet: Conn1, Conn2, U1, U2, U3, U4, U5
